Commit message: Fix right_hand_camera to be in right position, orientation, and in color

File: src/sawyer_robot/sawyer_description/urdf/sawyer_base.gazebo.xacro (robot description, xacro)
@@ -125,5 +125,5 @@
           <width>752</width>
           <height>480</height>
-          <format>L8</format>
+          <format>R8G8B8</format>
         </image>
         <clip>

File: src/sawyer_robot/sawyer_description/urdf/sawyer_base.urdf.xacro (robot description, xacro)
@@ -362,6 +362,6 @@
   <link name="right_hand_camera"/>
   <joint name="right_hand_camera" type="fixed">
-    <origin rpy="0 1.57079632679 0" xyz="0.039552 -0.033 0.0695"/>
-    <parent link="right_l5"/>
+    <origin rpy="0 0 0" xyz="0.0 -0.05 0.0"/>
+    <parent link="right_l6"/>
     <child link="right_hand_camera"/>
     <axis xyz="0 0 0"/>
