Commit message: correct head camera location to look down and be stationary

File: src/sawyer_robot/sawyer_description/urdf/sawyer_base.urdf.xacro (robot description, xacro)
@@ -527,6 +527,6 @@
   <link name="head_camera"/>
   <joint name="head_camera" type="fixed">
-    <origin rpy="-2.1293 0 -1.57079632679" xyz="0.0228027 0 0.216572"/>
-    <parent link="head"/>
+    <origin rpy="-2.8 -0.000 1.57079632679" xyz="1 0 0.593"/>
+    <parent link="base"/>
     <child link="head_camera"/>
     <axis xyz="0 0 0"/>

Commit message: move head camera

File: src/sawyer_robot/sawyer_description/urdf/sawyer_base.urdf.xacro (robot description, xacro)
@@ -527,5 +527,5 @@
   <link name="head_camera"/>
   <joint name="head_camera" type="fixed">
-    <origin rpy="-2.8 -0.000 1.57079632679" xyz="1 0 0.593"/>
+    <origin rpy="-2.4 -0.000 1.57079632679" xyz="1.3 0 0.35"/>
     <parent link="base"/>
     <child link="head_camera"/>
